File: ATTiny85-mppt.sch (KiCad schematic (older format))
At the start: 47 parts, among them J1 S+, J2 S-, J3 O+, J4 O-, Q1 BUK9511-55A127, Q2 BUK9511-55A127, Q4 2N2222A, Q5 2N2907A, SW1 Write OP-AMP DIFF, U1 LM7805_TO220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

Commit message: Fix by Invert Mode, 8Khz PWM. FET Bootstrap don't work with Higher frequency.
Parts:
- added Q3: 2N2222A, TO_SOT_Packages_THT:TO-92_Inline_Wide, symbol Device:Q_NPN_EBC
- added R9: 10k, Resistors_THT:R_Axial_DIN0309_L9.0mm_D3.2mm_P12.70mm_Horizontal, symbol Device:R
- Q5: value 2N2907A -> 2N2904A
Connections:
- net labels added: ~PWM
- net labels removed: PWM
- wire segments 190 -> 192
Other:
- moved on the sheet: Q4, R10, R7
Changed lines of the file:
@@
 Sheet 1 1
 Title "Simple MPPT with ATTiny85"
-Date "2018-10-30"
-Rev "1.2"
+Date "2018-10-31"
+Rev "1.3"
 Comp ""
 Comment1 ""
@@
 L Device:Q_NPN_EBC Q4
 U 1 1 55C35D82
-P 6500 2800
-F 0 "Q4" H 6800 2700 50  0000 R CNN
-F 1 "2N2222A" H 7000 2850 50  0000 R CNN
-F 2 "TO_SOT_Packages_THT:TO-92_Inline_Wide" H 6700 2900 29  0001 C CNN
-F 3 "" H 6500 2800 60  0000 C CNN
-	1    6500 2800
+P 6500 2900
+F 0 "Q4" H 6800 2800 50  0000 R CNN
+F 1 "2N2222A" H 7000 2950 50  0000 R CNN
+F 2 "TO_SOT_Packages_THT:TO-92_Inline_Wide" H 6700 3000 29  0001 C CNN
+F 3 "" H 6500 2900 60  0000 C CNN
+	1    6500 2900
 	1    0    0    -1
 $EndComp
@@
 L Device:R R10
 U 1 1 55C376F8
-P 5750 2700
-F 0 "R10" V 5830 2700 50  0000 C CNN
-F 1 "1k" V 5750 2700 50  0000 C CNN
-F 2 "Resistors_THT:R_Axial_DIN0309_L9.0mm_D3.2mm_P12.70mm_Horizontal" V 5680 2700 30  0001 C CNN
-F 3 "" H 5750 2700 30  0000 C CNN
-	1    5750 2700
-	0    1    1    0
+P 5450 2700
+F 0 "R10" V 5530 2700 50  0000 C CNN
+F 1 "1k" V 5450 2700 50  0000 C CNN
+F 2 "Resistors_THT:R_Axial_DIN0309_L9.0mm_D3.2mm_P12.70mm_Horizontal" V 5380 2700 30  0001 C CNN
+F 3 "" H 5450 2700 30  0000 C CNN
+	1    5450 2700
+	0    -1   -1   0
 $EndComp
 $Comp
@@
 Wire Wire Line
 	7650 2200 7750 2200
-Wire Wire Line
-	6600 3000 6600 3050
-Wire Wire Line
-	6600 3050 7450 3050
-Wire Wire Line
-	7450 3050 7450 2500
-Connection ~ 6600 3050
 Connection ~ 7750 2200
 Wire Wire Line
-	6300 2700 6300 2800
-Wire Wire Line
 	5400 2350 3500 2350
-Connection ~ 6300 2800
 Connection ~ 2250 2200
 Connection ~ 2650 5600
@@
 	8400 2200 8700 2200
 Wire Wire Line
-	6600 3050 6600 3100
-Wire Wire Line
 	7750 2200 7950 2200
 Wire Wire Line
-	6300 2800 6300 3300
-Wire Wire Line
 	2250 2200 2500 2200
 Wire Wire Line
@@
 Wire Wire Line
 	9500 2200 10000 2200
-Wire Wire Line
-	6700 5600 6400 5600
 Wire Wire Line
 	6700 4750 6700 5150
@@
 Text Notes 2000 6450 0    50   ~ 0
 Q1 rds <= 55milli Ohm. If bigger, R2/R3 and R4/R13 must change.
-Wire Wire Line
-	6300 2700 5900 2700
-Wire Wire Line
-	5300 2700 5600 2700
-Wire Wire Line
-	5300 2700 5300 3200
 $Comp
 L Device:R R7
 U 1 1 5BDAFBE4
-P 6250 2500
-F 0 "R7" V 6330 2500 50  0000 C CNN
-F 1 "1k" V 6250 2500 50  0000 C CNN
-F 2 "Resistors_THT:R_Axial_DIN0309_L9.0mm_D3.2mm_P12.70mm_Horizontal" V 6180 2500 30  0001 C CNN
-F 3 "" H 6250 2500 30  0000 C CNN
-	1    6250 2500
+P 6150 2750
+F 0 "R7" V 6230 2750 50  0000 C CNN
+F 1 "1k" V 6150 2750 50  0000 C CNN
+F 2 "Resistors_THT:R_Axial_DIN0309_L9.0mm_D3.2mm_P12.70mm_Horizontal" V 6080 2750 30  0001 C CNN
+F 3 "" H 6150 2750 30  0000 C CNN
+	1    6150 2750
 	0    1    1    0
 $EndComp
-Wire Wire Line
-	5700 2350 5850 2350
-Wire Wire Line
-	6400 2500 6600 2500
-Wire Wire Line
-	6600 2500 6600 2600
-Wire Wire Line
-	6100 2500 5850 2500
-Wire Wire Line
-	5850 2500 5850 2350
-Wire Wire Line
-	5850 2350 7150 2350
-Connection ~ 5850 2350
-Text Label 5350 2700 0    50   ~ 0
-PWM
+Text Label 5000 2650 0    50   ~ 0
+~PWM
 Wire Wire Line
 	7750 2200 7750 2950
@@
 	7150 2950 7150 2900
 Wire Wire Line
-	5200 5600 5650 5600
+	5200 5600 5400 5600
+$Comp
+L Device:Q_NPN_EBC Q3
+U 1 1 5BD9A966
+P 5800 3000
+F 0 "Q3" H 6100 2900 50  0000 R CNN
+F 1 "2N2222A" H 6300 3050 50  0000 R CNN
+F 2 "TO_SOT_Packages_THT:TO-92_Inline_Wide" H 6000 3100 29  0001 C CNN
+F 3 "" H 5800 3000 60  0000 C CNN
+	1    5800 3000
+	1    0    0    -1
+$EndComp
+Wire Wire Line
+	6100 5600 6700 5600
+Wire Wire Line
+	5300 2700 5300 3200
+Wire Wire Line
+	5600 2700 5600 3000
+Wire Wire Line
+	5900 3200 5900 3450
+Wire Wire Line
+	5900 3450 5750 3450
+Wire Wire Line
+	5750 3450 5750 3800
+Wire Wire Line
+	5750 3800 5400 3800
+Wire Wire Line
+	5400 3800 5400 5600
+Connection ~ 5400 5600
+Wire Wire Line
+	5400 5600 5650 5600
+$Comp
+L Device:R R9
+U 1 1 5BDD9D33
+P 5900 2600
+F 0 "R9" V 5980 2600 50  0000 C CNN
+F 1 "10k" V 5900 2600 50  0000 C CNN
+F 2 "Resistors_THT:R_Axial_DIN0309_L9.0mm_D3.2mm_P12.70mm_Horizontal" V 5830 2600 30  0001 C CNN
+F 3 "" H 5900 2600 30  0000 C CNN
+	1    5900 2600
+	-1   0    0    1
+$EndComp
+Wire Wire Line
+	5700 2350 5900 2350
+Wire Wire Line
+	5900 2750 5900 2800
+Wire Wire Line
+	5900 2350 5900 2450
+Connection ~ 5900 2350
+Wire Wire Line
+	5900 2350 6600 2350
+Wire Wire Line
+	6000 2750 5900 2750
+Connection ~ 5900 2750
+Wire Wire Line
+	6300 2750 6300 2900
 $Comp
 L Device:Q_PNP_EBC Q5
-U 1 1 55C35E2B
+U 1 1 5BE09576
 P 6500 3300
-F 0 "Q5" H 6800 3350 50  0000 R CNN
-F 1 "2N2907A" H 7000 3200 50  0000 R CNN
-F 2 "TO_SOT_Packages_THT:TO-92_Inline_Wide" H 6700 3400 29  0001 C CNN
-F 3 "" H 6500 3300 60  0000 C CNN
+F 0 "Q5" H 6691 3254 50  0000 L CNN
+F 1 "2N2904A" H 6691 3345 50  0000 L CNN
+F 2 "TO_SOT_Packages_THT:TO-92_Inline_Wide" H 6700 3400 50  0001 C CNN
+F 3 "~" H 6500 3300 50  0001 C CNN
 	1    6500 3300
 	1    0    0    1
 $EndComp
 Wire Wire Line
-	6400 4200 6400 5600
-Connection ~ 6400 5600
-Wire Wire Line
-	6400 5600 6100 5600
-Wire Wire Line
-	6600 3500 6600 4200
-Wire Wire Line
-	6600 4200 6400 4200
+	6300 3300 6300 2900
+Connection ~ 6300 2900
+Wire Wire Line
+	6600 3500 7750 3500
+Wire Wire Line
+	7750 3500 7750 2950
+Connection ~ 7750 2950
+Wire Wire Line
+	7450 2500 7450 3100
+Wire Wire Line
+	7450 3100 6600 3100
+Connection ~ 6600 3100
+Wire Wire Line
+	6600 2350 6600 2700
+Connection ~ 6600 2350
+Wire Wire Line
+	6600 2350 7150 2350
 $EndSCHEMATC

Commit message: fix FET bootstrap capacitor.
Parts:
- C2: value 1u -> >10uF
Changed lines of the file:
@@
 P 7150 2750
 F 0 "C2" H 7175 2850 50  0000 L CNN
-F 1 "1u" H 7175 2650 50  0000 L CNN
+F 1 ">10uF" H 7175 2650 50  0000 L CNN
 F 2 "Capacitors_THT:CP_Radial_D12.5mm_P5.00mm" H 7188 2600 30  0001 C CNN
 F 3 "" H 7150 2750 60  0000 C CNN

Commit message: Add another P FET for switching.
Parts:
- added Q6: BUK9508-55A, TO_SOT_Packages_THT-2:TO-220_Neutral123_Vertical, symbol Device:Q_PMOS_GDS
- added R17: 1M, Resistors_THT:R_Axial_DIN0309_L9.0mm_D3.2mm_P12.70mm_Horizontal, symbol Device:R
Connections:
- wire segments 192 -> 207
Other:
- moved on the sheet: C2, R10
Changed lines of the file:
@@
 Sheet 1 1
 Title "Simple MPPT with ATTiny85"
-Date "2018-10-31"
-Rev "1.3"
+Date "2018-11-02"
+Rev "1.4"
 Comp ""
 Comment1 ""
@@
 $EndComp
 $Comp
-L Device:Q_NMOS_GDS Q2
-U 1 1 55C35281
-P 7450 2300
-F 0 "Q2" V 7650 2550 50  0000 R CNN
-F 1 "BUK9511-55A127" V 7750 2600 50  0000 R CNN
-F 2 "TO_SOT_Packages_THT-2:TO-220_Neutral123_Vertical" H 7650 2400 29  0001 C CNN
-F 3 "" H 7450 2300 60  0000 C CNN
-	1    7450 2300
-	0    -1   -1   0
-$EndComp
-$Comp
 L 12f675-mppt-rescue:INDUCTOR L1
 U 1 1 55C35536
@@
 L Device:CP C2
 U 1 1 55C35FB2
-P 7150 2750
-F 0 "C2" H 7175 2850 50  0000 L CNN
-F 1 ">10uF" H 7175 2650 50  0000 L CNN
-F 2 "Capacitors_THT:CP_Radial_D12.5mm_P5.00mm" H 7188 2600 30  0001 C CNN
-F 3 "" H 7150 2750 60  0000 C CNN
-	1    7150 2750
+P 7050 2750
+F 0 "C2" H 7075 2850 50  0000 L CNN
+F 1 ">10uF" H 7075 2650 50  0000 L CNN
+F 2 "Capacitors_THT:CP_Radial_D12.5mm_P5.00mm" H 7088 2600 30  0001 C CNN
+F 3 "" H 7050 2750 60  0000 C CNN
+	1    7050 2750
 	1    0    0    -1
 $EndComp
@@
 L Device:R R10
 U 1 1 55C376F8
-P 5450 2700
-F 0 "R10" V 5530 2700 50  0000 C CNN
-F 1 "1k" V 5450 2700 50  0000 C CNN
-F 2 "Resistors_THT:R_Axial_DIN0309_L9.0mm_D3.2mm_P12.70mm_Horizontal" V 5380 2700 30  0001 C CNN
-F 3 "" H 5450 2700 30  0000 C CNN
-	1    5450 2700
-	0    -1   -1   0
+P 5450 2850
+F 0 "R10" V 5530 2850 50  0000 C CNN
+F 1 "1k" V 5450 2850 50  0000 C CNN
+F 2 "Resistors_THT:R_Axial_DIN0309_L9.0mm_D3.2mm_P12.70mm_Horizontal" V 5380 2850 30  0001 C CNN
+F 3 "" H 5450 2850 30  0000 C CNN
+	1    5450 2850
+	1    0    0    -1
 $EndComp
 $Comp
@@
 	9500 2200 9500 2350
 Wire Wire Line
-	7650 2200 7750 2200
+	7450 2200 7600 2200
 Connection ~ 7750 2200
 Wire Wire Line
@@
 Connection ~ 3750 3400
 Wire Wire Line
-	7150 2350 7150 2600
+	7050 2350 7050 2600
 Connection ~ 7400 5600
 Connection ~ 7400 4450
@@
 	8950 5100 8950 4850
 Wire Wire Line
-	7250 2200 3300 2200
+	7050 2200 6800 2200
 $Comp
 L Device:CP C7
@@
 	7750 2200 7750 2950
 Wire Wire Line
-	7750 2950 7150 2950
-Wire Wire Line
-	7150 2950 7150 2900
+	7750 2950 7050 2950
+Wire Wire Line
+	7050 2950 7050 2900
 Wire Wire Line
 	5200 5600 5400 5600
-$Comp
-L Device:Q_NPN_EBC Q3
-U 1 1 5BD9A966
-P 5800 3000
-F 0 "Q3" H 6100 2900 50  0000 R CNN
-F 1 "2N2222A" H 6300 3050 50  0000 R CNN
-F 2 "TO_SOT_Packages_THT:TO-92_Inline_Wide" H 6000 3100 29  0001 C CNN
-F 3 "" H 5800 3000 60  0000 C CNN
-	1    5800 3000
-	1    0    0    -1
-$EndComp
 Wire Wire Line
 	6100 5600 6700 5600
-Wire Wire Line
-	5300 2700 5300 3200
-Wire Wire Line
-	5600 2700 5600 3000
 Wire Wire Line
 	5900 3200 5900 3450
@@
 Connection ~ 7750 2950
 Wire Wire Line
-	7450 2500 7450 3100
-Wire Wire Line
-	7450 3100 6600 3100
+	7250 2500 7250 3100
+Wire Wire Line
+	7250 3100 6600 3100
 Connection ~ 6600 3100
 Wire Wire Line
@@
 Connection ~ 6600 2350
 Wire Wire Line
-	6600 2350 7150 2350
+	6600 2350 7050 2350
+$Comp
+L Device:Q_NMOS_GDS Q2
+U 1 1 5BDC3BBC
+P 7250 2300
+F 0 "Q2" V 7593 2300 50  0000 C CNN
+F 1 "BUK9511-55A127" V 7502 2300 50  0000 C CNN
+F 2 "TO_SOT_Packages_THT-2:TO-220_Neutral123_Vertical" H 7450 2400 50  0001 C CNN
+F 3 "~" H 7250 2300 50  0001 C CNN
+	1    7250 2300
+	0    -1   -1   0
+$EndComp
+$Comp
+L Device:Q_PMOS_GDS Q6
+U 1 1 5BDC4946
+P 7250 1700
+F 0 "Q6" V 7593 1700 50  0000 C CNN
+F 1 "BUK9508-55A" V 7502 1700 50  0000 C CNN
+F 2 "TO_SOT_Packages_THT-2:TO-220_Neutral123_Vertical" H 7450 1800 50  0001 C CNN
+F 3 "~" H 7250 1700 50  0001 C CNN
+	1    7250 1700
+	0    1    -1   0
+$EndComp
+Wire Wire Line
+	7050 1600 6800 1600
+Wire Wire Line
+	6800 1600 6800 2200
+Connection ~ 6800 2200
+Wire Wire Line
+	6800 2200 3300 2200
+Wire Wire Line
+	7450 1600 7600 1600
+Wire Wire Line
+	7600 1600 7600 2200
+Connection ~ 7600 2200
+Wire Wire Line
+	7600 2200 7750 2200
+$Comp
+L Device:Q_NPN_EBC Q3
+U 1 1 5BD9A966
+P 5800 3000
+F 0 "Q3" H 6100 2900 50  0000 R CNN
+F 1 "2N2222A" H 6300 3050 50  0000 R CNN
+F 2 "TO_SOT_Packages_THT:TO-92_Inline_Wide" H 6000 3100 29  0001 C CNN
+F 3 "" H 5800 3000 60  0000 C CNN
+	1    5800 3000
+	1    0    0    -1
+$EndComp
+Wire Wire Line
+	5300 3200 5300 2700
+Wire Wire Line
+	5300 2700 5450 2700
+Wire Wire Line
+	5450 3000 5600 3000
+Wire Wire Line
+	5600 3000 5600 2550
+Wire Wire Line
+	5600 2550 5750 2550
+Wire Wire Line
+	5750 2550 5750 1900
+Wire Wire Line
+	5750 1900 6100 1900
+Connection ~ 5600 3000
+$Comp
+L Device:R R17
+U 1 1 5BE61D3E
+P 6550 1600
+F 0 "R17" V 6630 1600 50  0000 C CNN
+F 1 "1M" V 6550 1600 50  0000 C CNN
+F 2 "Resistors_THT:R_Axial_DIN0309_L9.0mm_D3.2mm_P12.70mm_Horizontal" V 6480 1600 30  0001 C CNN
+F 3 "" H 6550 1600 30  0000 C CNN
+	1    6550 1600
+	0    -1   -1   0
+$EndComp
+Wire Wire Line
+	6700 1600 6800 1600
+Connection ~ 6800 1600
+Wire Wire Line
+	6400 1600 6100 1600
+Wire Wire Line
+	6100 1600 6100 1900
+Connection ~ 6100 1900
+Wire Wire Line
+	6100 1900 7250 1900
 $EndSCHEMATC

Commit message: Add AREF capacitor.
Parts:
- added C8: 10u, Capacitors_THT:CP_Radial_D12.5mm_P5.00mm, symbol Device:CP
Connections:
- wire segments 207 -> 211
Other:
- moved on the sheet: C5, R11
Changed lines of the file:
@@
 L Device:R R11
 U 1 1 55C4C21C
-P 6400 3600
-F 0 "R11" V 6480 3600 50  0000 C CNN
-F 1 "100k" V 6400 3600 50  0000 C CNN
-F 2 "Resistors_THT:R_Axial_DIN0309_L9.0mm_D3.2mm_P12.70mm_Horizontal" V 6330 3600 30  0001 C CNN
-F 3 "" H 6400 3600 30  0000 C CNN
-	1    6400 3600
+P 7300 3600
+F 0 "R11" V 7380 3600 50  0000 C CNN
+F 1 "100k" V 7300 3600 50  0000 C CNN
+F 2 "Resistors_THT:R_Axial_DIN0309_L9.0mm_D3.2mm_P12.70mm_Horizontal" V 7230 3600 30  0001 C CNN
+F 3 "" H 7300 3600 30  0000 C CNN
+	1    7300 3600
 	0    1    1    0
 $EndComp
@@
 L Device:CP C5
 U 1 1 55CDDBD9
-P 6100 4900
-F 0 "C5" H 6125 5000 50  0000 L CNN
-F 1 "10u" H 6125 4800 50  0000 L CNN
-F 2 "Capacitors_THT:CP_Radial_D12.5mm_P5.00mm" H 6138 4750 30  0001 C CNN
-F 3 "" H 6100 4900 60  0000 C CNN
-	1    6100 4900
+P 6200 4900
+F 0 "C5" H 6225 5000 50  0000 L CNN
+F 1 "10u" H 6225 4800 50  0000 L CNN
+F 2 "Capacitors_THT:CP_Radial_D12.5mm_P5.00mm" H 6238 4750 30  0001 C CNN
+F 3 "" H 6200 4900 60  0000 C CNN
+	1    6200 4900
 	1    0    0    -1
 $EndComp
@@
 Connection ~ 9500 2200
 Wire Notes Line
-	5900 5850 9800 5850
+	6050 5850 9800 5850
 Wire Wire Line
 	1850 4200 1850 5600
@@
 	5650 4050 6000 4050
 Wire Wire Line
-	6100 5050 6100 5600
-Connection ~ 6100 5600
-Wire Wire Line
-	6100 4750 6100 3600
-Connection ~ 6100 3600
-Wire Notes Line
-	5900 3500 5900 5850
-Wire Notes Line
-	5900 3500 6500 3500
+	6200 5050 6200 5600
+Connection ~ 6200 5600
+Wire Wire Line
+	6200 4750 6200 3600
+Connection ~ 6200 3600
+Wire Notes Line
+	6050 3500 6050 5850
+Wire Notes Line
+	6050 3500 6500 3500
 Wire Notes Line
 	6500 3500 6700 3750
@@
 	8850 3850 8850 3600
 Wire Wire Line
-	6550 3600 8850 3600
+	7450 3600 8850 3600
 Wire Wire Line
 	9450 4450 9450 4850
@@
 	8400 3950 8400 5200
 Wire Wire Line
-	6100 3600 6250 3600
+	6200 3600 7150 3600
 Wire Wire Line
 	5200 5600 4900 5600
@@
 	4450 2650 4450 2800
 Wire Wire Line
-	5400 3600 6100 3600
+	5400 3600 6200 3600
 Wire Wire Line
 	5300 3500 5050 3500
@@
 	5200 3400 5050 3400
 Wire Wire Line
-	5650 5600 6100 5600
+	5650 5600 5900 5600
 Wire Wire Line
 	5500 3100 5500 4500
@@
 	5200 5600 5400 5600
 Wire Wire Line
-	6100 5600 6700 5600
+	6200 5600 6700 5600
 Wire Wire Line
 	5900 3200 5900 3450
@@
 Wire Wire Line
 	6100 1900 7250 1900
+$Comp
+L Device:CP C8
+U 1 1 5BE62CB0
+P 5900 4900
+F 0 "C8" H 5925 5000 50  0000 L CNN
+F 1 "10u" H 5925 4800 50  0000 L CNN
+F 2 "Capacitors_THT:CP_Radial_D12.5mm_P5.00mm" H 5938 4750 30  0001 C CNN
+F 3 "" H 5900 4900 60  0000 C CNN
+	1    5900 4900
+	1    0    0    -1
+$EndComp
+Wire Wire Line
+	5900 4750 5900 4500
+Wire Wire Line
+	5900 4500 5650 4500
+Wire Wire Line
+	5900 5050 5900 5600
+Connection ~ 5900 5600
+Wire Wire Line
+	5900 5600 6200 5600
 $EndSCHEMATC

Commit message: remove some component.
Parts:
- removed Q6: BUK9508-55A, TO_SOT_Packages_THT-2:TO-220_Neutral123_Vertical, symbol Device:Q_PMOS_GDS
- removed R17: 1M, Resistors_THT:R_Axial_DIN0309_L9.0mm_D3.2mm_P12.70mm_Horizontal, symbol Device:R
- added D12: BZX 55c12(12V), Diodes_THT:D_DO-41_SOD81_P10.16mm_Horizontal, symbol Device:D_Zener
Connections:
- wire segments 211 -> 201
Changed lines of the file:
@@
 Sheet 1 1
 Title "Simple MPPT with ATTiny85"
-Date "2018-11-02"
-Rev "1.4"
+Date "2018-11-13"
+Rev "1.5"
 Comp ""
 Comment1 ""
@@
 Wire Wire Line
 	9500 2200 9500 2350
-Wire Wire Line
-	7450 2200 7600 2200
 Connection ~ 7750 2200
 Wire Wire Line
@@
 Wire Wire Line
 	8950 5100 8950 4850
-Wire Wire Line
-	7050 2200 6800 2200
 $Comp
 L Device:CP C7
@@
 	0    1    1    0
 $EndComp
-Text Label 5000 2650 0    50   ~ 0
+Text Label 5300 2700 0    50   ~ 0
 ~PWM
 Wire Wire Line
-	7750 2200 7750 2950
+	7750 2200 7750 2650
 Wire Wire Line
 	7750 2950 7050 2950
@@
 Connection ~ 7750 2950
 Wire Wire Line
-	7250 2500 7250 3100
+	7250 2500 7250 2650
 Wire Wire Line
 	7250 3100 6600 3100
@@
 $EndComp
 $Comp
-L Device:Q_PMOS_GDS Q6
-U 1 1 5BDC4946
-P 7250 1700
-F 0 "Q6" V 7593 1700 50  0000 C CNN
-F 1 "BUK9508-55A" V 7502 1700 50  0000 C CNN
-F 2 "TO_SOT_Packages_THT-2:TO-220_Neutral123_Vertical" H 7450 1800 50  0001 C CNN
-F 3 "~" H 7250 1700 50  0001 C CNN
-	1    7250 1700
-	0    1    -1   0
-$EndComp
-Wire Wire Line
-	7050 1600 6800 1600
-Wire Wire Line
-	6800 1600 6800 2200
-Connection ~ 6800 2200
-Wire Wire Line
-	6800 2200 3300 2200
-Wire Wire Line
-	7450 1600 7600 1600
-Wire Wire Line
-	7600 1600 7600 2200
-Connection ~ 7600 2200
-Wire Wire Line
-	7600 2200 7750 2200
-$Comp
 L Device:Q_NPN_EBC Q3
 U 1 1 5BD9A966
@@
 Wire Wire Line
 	5450 3000 5600 3000
-Wire Wire Line
-	5600 3000 5600 2550
-Wire Wire Line
-	5600 2550 5750 2550
-Wire Wire Line
-	5750 2550 5750 1900
-Wire Wire Line
-	5750 1900 6100 1900
-Connection ~ 5600 3000
-$Comp
-L Device:R R17
-U 1 1 5BE61D3E
-P 6550 1600
-F 0 "R17" V 6630 1600 50  0000 C CNN
-F 1 "1M" V 6550 1600 50  0000 C CNN
-F 2 "Resistors_THT:R_Axial_DIN0309_L9.0mm_D3.2mm_P12.70mm_Horizontal" V 6480 1600 30  0001 C CNN
-F 3 "" H 6550 1600 30  0000 C CNN
-	1    6550 1600
-	0    -1   -1   0
-$EndComp
-Wire Wire Line
-	6700 1600 6800 1600
-Connection ~ 6800 1600
-Wire Wire Line
-	6400 1600 6100 1600
-Wire Wire Line
-	6100 1600 6100 1900
-Connection ~ 6100 1900
-Wire Wire Line
-	6100 1900 7250 1900
 $Comp
 L Device:CP C8
@@
 Wire Wire Line
 	5900 5600 6200 5600
+$Comp
+L Device:D_Zener D12
+U 1 1 5BEB0C16
+P 7500 2650
+F 0 "D12" H 7500 2866 50  0000 C CNN
+F 1 "BZX 55c12(12V)" H 7500 2775 50  0000 C CNN
+F 2 "Diodes_THT:D_DO-41_SOD81_P10.16mm_Horizontal" H 7500 2650 50  0001 C CNN
+F 3 "~" H 7500 2650 50  0001 C CNN
+	1    7500 2650
+	1    0    0    -1
+$EndComp
+Wire Wire Line
+	7650 2650 7750 2650
+Connection ~ 7750 2650
+Wire Wire Line
+	7750 2650 7750 2950
+Wire Wire Line
+	7350 2650 7250 2650
+Connection ~ 7250 2650
+Wire Wire Line
+	7250 2650 7250 3100
+Wire Wire Line
+	3300 2200 7050 2200
+Wire Wire Line
+	7450 2200 7750 2200
 $EndSCHEMATC

Commit message: update bootstrap capacitor.
Parts:
- C2: value >10uF -> 47uF 50v
Changed lines of the file:
@@
 P 7050 2750
 F 0 "C2" H 7075 2850 50  0000 L CNN
-F 1 ">10uF" H 7075 2650 50  0000 L CNN
+F 1 "47uF 50v" H 7075 2650 50  0000 L CNN
 F 2 "Capacitors_THT:CP_Radial_D12.5mm_P5.00mm" H 7088 2600 30  0001 C CNN
 F 3 "" H 7050 2750 60  0000 C CNN

Commit message: update PCB file. update capacitor and add resistor.
Parts:
- added R17: 1k, Resistors_THT:R_Axial_DIN0309_L9.0mm_D3.2mm_P2.54mm_Vertical, symbol Device:R
- C2: value 47uF 50v -> 22uF 50v
Connections:
- wire segments 201 -> 202
Changed lines of the file:
@@
 Sheet 1 1
 Title "Simple MPPT with ATTiny85"
-Date "2018-11-13"
-Rev "1.5"
+Date "2018-11-17"
+Rev "1.6"
 Comp ""
 Comment1 ""
@@
 P 7050 2750
 F 0 "C2" H 7075 2850 50  0000 L CNN
-F 1 "47uF 50v" H 7075 2650 50  0000 L CNN
+F 1 "22uF 50v" H 7075 2650 50  0000 L CNN
 F 2 "Capacitors_THT:CP_Radial_D12.5mm_P5.00mm" H 7088 2600 30  0001 C CNN
 F 3 "" H 7050 2750 60  0000 C CNN
@@
 	7250 2500 7250 2650
 Wire Wire Line
-	7250 3100 6600 3100
-Connection ~ 6600 3100
-Wire Wire Line
 	6600 2350 6600 2700
 Connection ~ 6600 2350
@@
 Wire Wire Line
 	7450 2200 7750 2200
+$Comp
+L Device:R R17
+U 1 1 5BF0956D
+P 6950 3100
+F 0 "R17" V 7030 3100 50  0000 C CNN
+F 1 "1k" V 6950 3100 50  0000 C CNN
+F 2 "Resistors_THT:R_Axial_DIN0309_L9.0mm_D3.2mm_P2.54mm_Vertical" V 6880 3100 30  0001 C CNN
+F 3 "" H 6950 3100 30  0000 C CNN
+	1    6950 3100
+	0    1    1    0
+$EndComp
+Wire Wire Line
+	7250 3100 7100 3100
+Wire Wire Line
+	6800 3100 6600 3100
+Connection ~ 6600 3100
 $EndSCHEMATC

Commit message: fix Q5 value.
Parts:
- Q5: value 2N2904A -> 2N2907A
Changed lines of the file:
@@
 P 6500 3300
 F 0 "Q5" H 6691 3254 50  0000 L CNN
-F 1 "2N2904A" H 6691 3345 50  0000 L CNN
+F 1 "2N2907A" H 6691 3345 50  0000 L CNN
 F 2 "TO_SOT_Packages_THT:TO-92_Inline_Wide" H 6700 3400 50  0001 C CNN
 F 3 "~" H 6500 3300 50  0001 C CNN
