File: ATTiny85-mppt.sch (KiCad schematic (older format))
At the start: 52 parts, among them J1 S+, J2 S-, J3 O+, J4 O-, Q1 BUK9511-55A127, Q2 BUK9511-55A127, Q3 2N2222A, Q4 2N2222A, Q5 2N2907A, SW1 Write OP-AMP DIFF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

Commit message: R11 to 4.7k
Parts:
- R11: value 100k -> 4.7k
Changed lines of the file:
@@
 P 7300 3600
 F 0 "R11" V 7380 3600 50  0000 C CNN
-F 1 "100k" V 7300 3600 50  0000 C CNN
+F 1 "4.7k" V 7300 3600 50  0000 C CNN
 F 2 "Resistors_THT:R_Axial_DIN0309_L9.0mm_D3.2mm_P12.70mm_Horizontal" V 7230 3600 30  0001 C CNN
 F 3 "" H 7300 3600 30  0000 C CNN

Commit message: Remove R11. It is a lot lower current sensing voltage.
Parts:
- removed R11: 4.7k, Resistors_THT:R_Axial_DIN0309_L9.0mm_D3.2mm_P12.70mm_Horizontal, symbol Device:R
Connections:
- wire segments 202 -> 201
Changed lines of the file:
@@
 Sheet 1 1
 Title "Simple MPPT with ATTiny85"
-Date "2018-11-17"
-Rev "1.6"
+Date "2018-11-29"
+Rev "1.7"
 Comp ""
 Comment1 ""
@@
 Heat Sink
 $Comp
-L Device:R R11
-U 1 1 55C4C21C
-P 7300 3600
-F 0 "R11" V 7380 3600 50  0000 C CNN
-F 1 "4.7k" V 7300 3600 50  0000 C CNN
-F 2 "Resistors_THT:R_Axial_DIN0309_L9.0mm_D3.2mm_P12.70mm_Horizontal" V 7230 3600 30  0001 C CNN
-F 3 "" H 7300 3600 30  0000 C CNN
-	1    7300 3600
-	0    1    1    0
-$EndComp
-$Comp
 L Device:R R12
 U 1 1 55C48C57
@@
 	8850 3850 8850 3600
 Wire Wire Line
-	7450 3600 8850 3600
-Wire Wire Line
 	9450 4450 9450 4850
 Connection ~ 8400 5600
@@
 Wire Wire Line
 	8400 3950 8400 5200
-Wire Wire Line
-	6200 3600 7150 3600
 Wire Wire Line
 	4300 4400 5300 4400
@@
 Wire Wire Line
 	5050 3100 5500 3100
+Wire Wire Line
+	6200 3600 8850 3600
 $EndSCHEMATC

Commit message: update circuit.
Parts:
- removed R17: 1k, Resistors_THT:R_Axial_DIN0309_L9.0mm_D3.2mm_P2.54mm_Vertical, symbol Device:R
Connections:
- wire segments 201 -> 200
Changed lines of the file:
@@
 Wire Wire Line
 	7450 2200 7750 2200
-$Comp
-L Device:R R17
-U 1 1 5BF0956D
-P 6950 3100
-F 0 "R17" V 7030 3100 50  0000 C CNN
-F 1 "1k" V 6950 3100 50  0000 C CNN
-F 2 "Resistors_THT:R_Axial_DIN0309_L9.0mm_D3.2mm_P2.54mm_Vertical" V 6880 3100 30  0001 C CNN
-F 3 "" H 6950 3100 30  0000 C CNN
-	1    6950 3100
-	0    1    1    0
-$EndComp
-Wire Wire Line
-	7250 3100 7100 3100
-Wire Wire Line
-	6800 3100 6600 3100
 Connection ~ 6600 3100
 Wire Wire Line
@@
 Wire Wire Line
 	6200 3600 8850 3600
+Wire Wire Line
+	6600 3100 7250 3100
 $EndSCHEMATC

Commit message: update.
Other:
- note added: "D12, C8 - optional"
Changed lines of the file:
@@
 Wire Wire Line
 	6600 3100 7250 3100
+Text Notes 2000 6800 0    50   ~ 0
+D12, C8 - optional
 $EndSCHEMATC

Commit message: update C2 value. 10uF is also good.
Parts:
- C2: value 22uF 50v -> 22uF(or 10uF) 50v
Changed lines of the file:
@@
 P 7050 2750
 F 0 "C2" H 7075 2850 50  0000 L CNN
-F 1 "22uF 50v" H 7075 2650 50  0000 L CNN
+F 1 "22uF(or 10uF) 50v" H 7075 2650 50  0000 L CNN
 F 2 "Capacitors_THT:CP_Radial_D12.5mm_P5.00mm" H 7088 2600 30  0001 C CNN
 F 3 "" H 7050 2750 60  0000 C CNN

Commit message: C6 to optional component.
Other:
- note added: "D12, C8, C6 - optional"
- note removed: "D12, C8 - optional"
Changed lines of the file:
@@
 U 1 1 55D02AF9
 P 4300 5000
-F 0 "C6" H 4200 5250 50  0000 L CNN
-F 1 "10u" H 4100 5150 50  0000 L CNN
+F 0 "C6" H 4150 4900 50  0000 L CNN
+F 1 "10u" H 4150 4800 50  0000 L CNN
 F 2 "Capacitors_THT:CP_Radial_D12.5mm_P5.00mm" H 4338 4850 30  0001 C CNN
 F 3 "" H 4300 5000 60  0000 C CNN
@@
 	6600 3100 7250 3100
 Text Notes 2000 6800 0    50   ~ 0
-D12, C8 - optional
+D12, C8, C6 - optional
 $EndSCHEMATC

Commit message: Low voltage-High current stuck solved by removing C6. More testing.
Other:
- note added: "C6 - It is bad for power calculation. Remove it."
- note added: "D12, C8 - optional"
- note removed: "D12, C8, C6 - optional"
Changed lines of the file:
@@
 	6600 3100 7250 3100
 Text Notes 2000 6800 0    50   ~ 0
-D12, C8, C6 - optional
+D12, C8 - optional
+Text Notes 2000 6900 0    50   ~ 0
+C6 - It is bad for power calculation. Remove it.
 $EndSCHEMATC

Commit message: Remove C6
Parts:
- removed C6: 10u, Capacitors_THT:CP_Radial_D12.5mm_P5.00mm, symbol Device:CP
Connections:
- wire segments 200 -> 196
Other:
- note removed: "C6 - It is bad for power calculation. Remove it."
Changed lines of the file:
@@
 Sheet 1 1
 Title "Simple MPPT with ATTiny85"
-Date "2018-11-29"
-Rev "1.7"
+Date "2018-12-17"
+Rev "1.8"
 Comp ""
 Comment1 ""
@@
 	1    0    0    -1
 $EndComp
-$Comp
-L Device:CP C6
-U 1 1 55D02AF9
-P 4300 5000
-F 0 "C6" H 4150 4900 50  0000 L CNN
-F 1 "10u" H 4150 4800 50  0000 L CNN
-F 2 "Capacitors_THT:CP_Radial_D12.5mm_P5.00mm" H 4338 4850 30  0001 C CNN
-F 3 "" H 4300 5000 60  0000 C CNN
-	1    4300 5000
-	1    0    0    -1
-$EndComp
 Text Label 8550 6000 0    60   ~ 0
 3.6v
@@
 	4550 4300 4550 4750
 Wire Wire Line
-	4300 5150 4300 5600
-Connection ~ 4300 5600
-Wire Wire Line
 	2100 3500 2100 4400
 Wire Wire Line
 	2100 4400 3700 4400
-Wire Wire Line
-	4000 4400 4300 4400
-Wire Wire Line
-	4300 4850 4300 4400
-Connection ~ 4300 4400
 Wire Wire Line
 	5650 4500 5500 4500
@@
 	1850 3500 1850 3900
 Wire Wire Line
-	4550 5600 4300 5600
-Wire Wire Line
 	3100 4000 3750 4000
 Wire Wire Line
@@
 Wire Wire Line
 	8400 3950 8400 5200
-Wire Wire Line
-	4300 4400 5300 4400
 Wire Wire Line
 	5650 4500 5650 4650
@@
 	4550 5600 5400 5600
 Wire Wire Line
-	4300 5600 2650 5600
-Wire Wire Line
 	2150 3100 3300 3100
 Wire Wire Line
@@
 Text Notes 2000 6800 0    50   ~ 0
 D12, C8 - optional
-Text Notes 2000 6900 0    50   ~ 0
-C6 - It is bad for power calculation. Remove it.
+Wire Wire Line
+	2650 5600 4550 5600
+Wire Wire Line
+	4000 4400 5300 4400
 $EndSCHEMATC
