File: ATTiny85-mppt.kicad_pcb (KiCad board)
At the start: 2 copper layers, 97.6 x 90.8 mm, 55 parts, among them Q1 BUK9511-55A127, Q2 BUK9511-55A127, Q3 2N2222A, Q4 2N2222A, Q5 2N2907A, Q6 2N2222A, Q7 2N2222A, U1 LM7805_TO220, U2 LM358N, U3 ATtiny85-20PU

Commit message: update PCB.
Parts:
- added C8: 10u, Capacitors_THT:CP_Radial_D12.5mm_P5.00mm, F.Cu at (57.9, 81.2)
- R1: value 47k -> 2.2k
- R11: value 33k -> 10k
- R15: value 1k -> 2.2k
- R2, R4: value 200k -> 100k
- moved R11 42.1 mm to (108.0, 70.1)
- moved R15 37.8 mm to (71.5, 76.9), turned to 0 degrees
- moved R1 23.6 mm to (71.5, 93.9), turned to 90 degrees
- moved R2 21.4 mm to (78.7, 94.0)
- moved R3 16.9 mm to (90.3, 91.9), turned to 90 degrees
- moved R13 5.66 mm to (83.5, 94.0), turned to 90 degrees
- moved D8 5.29 mm to (103.7, 83.6), turned to 90 degrees
- moved R4 5.01 mm to (95.1, 79.2), turned to 270 degrees
- moved D9 4.65 mm to (103.7, 89.5), turned to 90 degrees
- moved R14 3.20 mm to (103.7, 64.3)
- moved C1 1.69 mm to (96.6, 98.8)
Connections:
- D8 pad 1: /1.8v -> Net-(D8-Pad1)
- D9 pad 2: /1.8v -> Net-(D8-Pad1)
- Q1 pad 1: Net-(Q1-Pad1) -> /3.6v
- R1 pad 1: /BootStrap -> GND
- R1 pad 2: /2.06v -> Net-(R1-Pad2)
- R11 pad 1: GND -> /BootStrap
- R11 pad 2: /2.06v -> /~PWM
- R15 pad 1: Net-(R15-Pad1) -> Net-(R1-Pad2)
- R15 pad 2: /1.8v -> /PV-Current
- R4 pad 1: /PV-Current -> Net-(R4-Pad1)
- U2 pad 1: Net-(Q1-Pad1) -> /PV-Current
- U2 pad 2: Net-(R15-Pad1) -> Net-(R1-Pad2)
- U2 pad 3: /2.06v -> Net-(R4-Pad1)
- U2 pad 7: /PV-Current -> Net-(R4-Pad1)
Routing:
- net /3.6v: track 35.3 -> 109.8 mm
- net Net-(Q1-Pad1): track 46.7 -> 0.00 mm
- net /2.06v: track 39.7 -> 0.00 mm
- net /BootStrap: track 123.2 -> 89.1 mm
- net Net-(R1-Pad2): track 0.00 -> 28.9 mm
- net Net-(R15-Pad1): track 21.6 -> 0.00 mm
- net Net-(R4-Pad1): track 0.00 -> 21.5 mm
- net PRI_LO: track 166.0 -> 149.2 mm
- net Net-(R13-Pad2): track 19.3 -> 29.8 mm
- net /1.8v: track 10.1 -> 0.00 mm
- net Net-(R6-Pad2): track 47.5 -> 52.6 mm
- net GND: track 369.2 -> 373.7 mm
- net /PV-Current: track 58.7 -> 54.9 mm
- net Net-(D8-Pad1): track 0.00 -> 3.30 mm
- net /~PWM: track 9.97 -> 13.1 mm
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Other:
- board text added: "MPPT 1.92"
- board text removed: "MPPT 2.0"

Commit message: Update PCB files.
Connections:
- net /~PWM renamed /~{PWM}
Other:
- net class Default removed
